File: hardware/tactigotchi.kicad_pcb (KiCad board)
At the start: 2 copper layers, 70.5 x 39.9 mm, 41 parts, among them Q1 BC817, Q2 BC817, SW1 SW_Push, SW2 SW_Push, SW3 SW_Push, SW4 SW_Push, SW5 SW_Push, SW6 SW_Push, SW7 SW_Push, SW8 SW_Push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

Commit message: Add files via upload
Parts:
- BT1, C10, C11, C12, C2, C6, C7, C8, C9, L1, R10, R2, R5, R6, R7, R8, R9, U2, U4, U5: moved to B.Cu
- C5: moved to F.Cu
- moved C10 124.5 mm to (63.0, 149.6), turned to -90 degrees
- moved R2 120.5 mm to (76.4, 146.8)
- moved C9 119.6 mm to (67.8, 154.1), turned to 180 degrees
- moved C8 111.1 mm to (76.3, 151.0), turned to 180 degrees
- moved U2 109.2 mm to (69.2, 149.3), turned to 180 degrees
- moved R11 80.6 mm to (138.3, 78.4)
- moved C6 80.3 mm to (76.4, 111.2), turned to 90 degrees
- moved C7 79.3 mm to (76.4, 117.1), turned to 90 degrees
- moved LS1 74.2 mm to (56.4, 152.4), turned to 90 degrees
- moved D1 74.0 mm to (139.4, 63.6)
- moved Q1 70.1 mm to (138.3, 73.6), turned to 0 degrees
- moved R1 70.0 mm to (138.4, 68.7)
- moved R7 62.5 mm to (72.4, 111.2), turned to -90 degrees
- moved C12 60.9 mm to (135.4, 110.4), turned to -90 degrees
- moved C11 59.7 mm to (139.9, 110.4), turned to -90 degrees
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Connections:
- U1 pad 10: unconnected-(U1-NC-Pad10) -> GND
- U1 pad 11: unconnected-(U1-NC-Pad11) -> GND
- U1 pad 12: unconnected-(U1-NC-Pad12) -> GND
- U1 pad 13: unconnected-(U1-NC-Pad13) -> GND
- U1 pad 14: unconnected-(U1-NC-Pad14) -> GND
Routing:
- net /PSU_3v3: track 0.00 -> 210.0 mm, vias 0 -> 4
- net /3v3_MCU: track 0.00 -> 121.8 mm
- net /LCD_LED_CTL: track 0.00 -> 117.8 mm
- net /SPI0_MISO: track 0.00 -> 115.8 mm, vias 0 -> 2
- net Net-(A1-GPIO2): track 0.00 -> 110.7 mm, vias 0 -> 1
- net /SPI0_MOSI: track 0.00 -> 104.5 mm, vias 0 -> 1
- net /SPI0_SCLK: track 0.00 -> 103.9 mm, vias 0 -> 1
- net Net-(A1-GPIO4): track 0.00 -> 100.6 mm, vias 0 -> 1
- net /CS_LCD: track 0.00 -> 95.4 mm, vias 0 -> 1
- net Net-(A1-GPIO3): track 0.00 -> 89.4 mm, vias 0 -> 1
- net /DC_LCD: track 0.00 -> 87.4 mm, vias 0 -> 2
- net /RST_LCD: track 0.00 -> 86.5 mm
- net Net-(A1-GPIO5): track 0.00 -> 84.9 mm, vias 0 -> 1
- net /IR_LED_CTL: track 0.00 -> 79.4 mm
- net /PSU_EN: track 0.00 -> 79.0 mm, vias 0 -> 2
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- added copper zone on B.Cu, net GND
- added copper zone on F.Cu, net GND
Other:
- board size 70.5 x 39.9 mm -> 97.4 x 97.7 mm
